Commit message: World added

File: install/rmitbot_description/share/rmitbot_description/urdf/rmitbot_laser.xacro (robot description, xacro)
@@ -9,5 +9,5 @@
         </inertial>
         <visual>
-            <origin xyz="0 0 0" rpy="0 0 0" />
+            <origin xyz="0 0 0" rpy="0 0 3.14" />
             <geometry>
                 <mesh filename="package://rmitbot_description/meshes/laser_link.STL" />
@@ -22,5 +22,5 @@
     </link>
     <joint name="laser_joint" type="fixed">
-        <origin xyz="0. 0. 0.14" rpy="0 0 3.14" />
+        <origin xyz="0. 0. 0.14" rpy="0 0 0" />
         <parent link="base_link" />
         <child link="laser_link" />
